Commit message: Add build and install files for roomba_description package

File: src/robot_description/urdf/ZavaQuin.urdf (robot description, URDF)
Before this commit: robot ZavaQuin, 7 links, 6 joints
Links:
- added link base_footprint, mass 0.001; collision box size=0.001 0.001 0.001; visual box size=0.001 0.001 0.001
Joints:
- added joint base_footprint_to_base_link: type fixed, parent base_footprint, child base_link, origin xyz=0 0 0 rpy=0 0 0
