Commit message: gazebo

File: zavaquin_description/urdf/camera.xacro (robot description, xacro)
@@ -1,4 +1,7 @@
 <?xml version="1.0" ?>
 <robot xmlns:xacro="http://ros.org/wiki/xacro">
+    <material name="purple">
+        <color rgba="0.54117647058 0.54117647058 0.7294117647 1.0" />
+    </material>
     <!-- Camera -->
     <link name="camera_link">
@@ -19,7 +22,5 @@
                 <mesh filename="package://zavaquin_description/meshes/camera_link.STL" />
             </geometry>
-            <material name="">
-                <color rgba="0.866666666666667 0.909803921568627 1 1" />
-            </material>
+            <material name="purple" />
         </visual>
         <collision>
@@ -33,5 +34,5 @@
     <parent link="base_link"/>
     <child link="camera_link"/>
-    <origin xyz="0.00039991 -0.17103 0.097276" rpy="0 0 {-pi/2}"/>
+    <origin xyz="0.00039991 -0.17103 0.097276" rpy="0 0 ${-pi/2}"/>
     <axis xyz="0 0 0"/>
   </joint>

File: zavaquin_description/urdf/imu.xacro (robot description, xacro)
@@ -19,6 +19,6 @@
                 <mesh filename="package://zavaquin_description/meshes/imu_link.STL" />
             </geometry>
-            <material name="">
-                <color rgba="0.827450980392157 0.83921568627451 0.827450980392157 1" />
+            <material name="dark">
+                <color rgba="0.01960784313 0.01960784313 0.01960784313 0.8" />
             </material>
         </visual>
@@ -33,5 +33,5 @@
         <parent link="base_link"/>
         <child link="imu_link"/>
-        <origin xyz="-0.0390281436839592 0.0549871759093349 0.010774999999999" rpy="0 0 {-pi/2}"/>
+        <origin xyz="-0.0390281436839592 0.0549871759093349 0.010774999999999" rpy="0 0 ${-pi/2}"/>
         <axis xyz="0 0 0" />
     </joint>

File: zavaquin_description/urdf/lidar.xacro (robot description, xacro)
@@ -18,6 +18,6 @@
               <mesh filename="package://zavaquin_description/meshes/laser_link.STL" />
             </geometry>
-            <material name="">
-              <color rgba="0.792156862745098 0.819607843137255 0.933333333333333 1" />
+            <material name="dark">
+                <color rgba="0.01960784313 0.01960784313 0.01960784313 0.8" />
             </material>
         </visual>

File: zavaquin_description/urdf/ros2_control.xacro (robot description, xacro)
@@ -55,5 +55,5 @@
         <plugin>gazebo_ros2_control/GazeboSystem</plugin>
       </hardware>
-      <joint name='left_wheel_joint'>
+      <joint name='wheel_left_joint'>
         <command_interface name='velocity'>
           <param name='min'>-10</param>
@@ -63,5 +63,5 @@
         <state_interface name='position'/>
       </joint>
-      <joint name='right_wheel_joint'>
+      <joint name='wheel_right_joint'>
         <command_interface name='velocity'>
           <param name='min'>-10</param>

File: zavaquin_description/urdf/zavaquin.urdf.xacro (robot description, xacro)
@@ -6,4 +6,10 @@
   <xacro:arg name="use_ros2_control" default="true"/>
   <xacro:arg name="sim_mode" default="false"/>
+  <material name="dark">
+    <color rgba="0.01960784313 0.01960784313 0.01960784313 1.0" />
+  </material>
+  <material name="red">
+    <color rgba="0.89019607843 0.14509803921 0.12156862745 1.0" />
+  </material>
   <link name="base_footprint"/>
   <joint name="base_footprint_to_base_link" type="fixed">
@@ -29,7 +35,5 @@
         <mesh filename="package://zavaquin_description/meshes/base_link.STL" />
       </geometry>
-      <material name="">
-        <color rgba="0.749019607843137 0.749019607843137 0.749019607843137 1" />
-      </material>
+      <material name="red" />
     </visual>
     <collision>
@@ -57,7 +61,5 @@
         <mesh filename="package://zavaquin_description/meshes/wheel_left_link.STL" />
       </geometry>
-      <material name="">
-        <color rgba="0.792156862745098 0.819607843137255 0.933333333333333 1" />
-      </material>
+      <material name="dark" />
     </visual>
     <collision>
@@ -91,7 +93,5 @@
         <mesh filename="package://zavaquin_description/meshes/wheel_right_link.STL" />
       </geometry>
-      <material name="">
-        <color rgba="0.792156862745098 0.819607843137255 0.933333333333333 1" />
-      </material>
+      <material name="dark" />
     </visual>
     <collision>
@@ -125,7 +125,5 @@
         <mesh filename="package://zavaquin_description/meshes/caster_wheel_link.STL" />
       </geometry>
-      <material name="">
-        <color rgba="0.749019607843137 0.749019607843137 0.749019607843137 1" />
-      </material>
+      <material name="dark" />
     </visual>
     <collision>
@@ -156,5 +154,5 @@
     <maxVel>0.1</maxVel>
     <fdir1>1 0 0</fdir1>
-    <material>Gazebo/FlatBlack</material>
+    <material>Gazebo/Flatdark</material>
   </gazebo>
   <gazebo reference="wheel_right_link">
@@ -166,10 +164,10 @@
     <maxVel>0.1</maxVel>
     <fdir1>1 0 0</fdir1>
-    <material>Gazebo/FlatBlack</material>
+    <material>Gazebo/Flatdark</material>
   </gazebo>
   <gazebo reference="caster_wheel_link">
     <mu1>0.1</mu1>
     <mu2>0.1</mu2>
-    <material>Gazebo/FlatBlack</material>
+    <material>Gazebo/Flatdark</material>
   </gazebo>
   <xacro:if value="$(arg use_ros2_control)">
