Commit message: actualizacion3

File: zavaquin_description/urdf/ros2_control.xacro (robot description, xacro)
@@ -6,10 +6,10 @@
       <hardware>
         <plugin>lidarbot_base/LidarbotHardware</plugin>
-          <param name='left_wheel_name'>left_wheel_joint</param>
-          <param name='right_wheel_name'>right_wheel_joint</param>
+          <param name='left_wheel_name'>wheel_left_joint</param>
+          <param name='right_wheel_name'>wheel_right_joint</param>
 	  <param name='enc_ticks_per_rev'>1084</param>
           <param name='loop_rate'>30.0</param>
       </hardware>
-      <joint name='left_wheel_joint'>
+      <joint name='wheel_left_joint'>
         <command_interface name='velocity'>
           <param name='min'>-10</param>
@@ -19,5 +19,5 @@
         <state_interface name='position'/>
       </joint>
-      <joint name='right_wheel_joint'>
+      <joint name='wheel_right_joint'>
         <command_interface name='velocity'>
           <param name='min'>-10</param>
@@ -27,24 +27,4 @@
         <state_interface name='position'/>
       </joint>
-    </ros2_control>
-    <!-- MPU6050 sensor-->
-    <ros2_control name='MPU6050' type='sensor'>
-      <hardware>
-        <plugin>lidarbot_bringup/MPU6050Hardware</plugin>
-          <param name='sensor_name'>mpu6050</param>
-          <param name='frame_id'>imu_link</param>
-      </hardware>
-      <sensor name='mpu6050'>
-        <state_interface name='orientation.x'/>
-        <state_interface name='orientation.y'/>
-        <state_interface name='orientation.z'/>
-        <state_interface name='orientation.w'/>
-        <state_interface name='angular_velocity.x'/>
-        <state_interface name='angular_velocity.y'/>
-        <state_interface name='angular_velocity.z'/>
-        <state_interface name='linear_acceleration.x'/>
-        <state_interface name='linear_acceleration.y'/>
-        <state_interface name='linear_acceleration.z'/>
-      </sensor>
     </ros2_control>
   </xacro:unless>
